Commit message: 单一机械臂控制测试通过

File: src/frcobot_ros/frcobot_description/urdf/fr5v6.urdf (robot description, URDF)
Before this commit: robot fr5v6, 9 links, 8 joints
Links:
- removed link tool_Link
Joints:
- removed joint tool

File: src/frcobot_ros/frcobot_description/urdf/fr5v6_gazebo.urdf (robot description, URDF)
Before this commit: robot fr5v6, 9 links, 8 joints
Links:
- removed link tool_Link
Joints:
- removed joint tool
